File: Hardware/B_PSU_0x00.kicad_pcb (KiCad board)
At the start: 2 copper layers, 72.5 x 55 mm, 78 parts, among them J1 Conn_01x03, J10 Conn_01x02, J12 Conn_01x03, J13 Conn_01x03, J14 Conn_01x02, J15 Conn_01x02, J16 Conn_01x02, J17 Conn_01x02, J18 Conn_01x03, J19 Conn_01x03, J2 Conn_01x02, J20 Conn_01x03, J21 Conn_01x03, J22 Conn_01x03, J23 Conn_01x02, J24 Conn_01x02, J25 Conn_01x02, J26 Conn_01x02, J27 Conn_01x03, J28 Conn_01x03, J6 Conn_01x03, J7 Conn_01x02, J8 Conn_01x02, J9 Conn_01x02, U1 ADP5070AREZ, U2 ADP7118WAUJZ-5.0, U3 ADP7118AUJZ-3.3-R7, U4 ADP7142AUJZ-1.8, U5 ADP7118AUJZ-2.5-R7, U6 ADP7182ACPZ-5.0-R7, U7 ADP7183ACPZN3.3-R7, U8 ADP7182ACPZN-2.5R7, U9 ADP7182AUJZ-1.8

Commit message: 0x00 version and revision files for manufacturing
Parts:
- moved Creg1 8.94 mm to (114.3, 78.2)
- moved Ca1 7.54 mm to (125.2, 77.7), turned to 90 degrees
- moved Cafb1 4.16 mm to (122.4, 77.7), turned to 90 degrees
- moved U9 0.94 mm to (110.7, 52.1), turned to 90 degrees
- moved U7 0.59 mm to (118.6, 77.7)
- moved U4 0.53 mm to (119.4, 52.1), turned to 90 degrees
- moved U5 0.25 mm to (102.4, 52.1), turned to 0 degrees
- moved Cout6 0.14 mm to (96.3, 48.5)
Connections:
- Ca1 pad 1: Net-(U7-VA) -> /Va
- Cafb1 pad 1: Net-(U7-VA) -> /Va
- Cafb1 pad 2: Net-(U7-VAFB) -> /Vafb
- Cout4 pad 2: Net-(J12-Pin_3) -> /-3v3
- Creg1 pad 1: Net-(U7-VREG) -> /Vreg
- J12 pad 3: Net-(J12-Pin_3) -> /-3v3
- J19 pad 3: Net-(J12-Pin_3) -> /-3v3
- U7 pad 3: (no net) -> /Va
- U7 pad 4: (no net) -> /Vafb
- U7 pad 6: Net-(Cin3-Pad2) -> /GND_3v3
- U7 pad 7: (no net) -> /Vreg
- U7 pad 8: Net-(Cin4-Pad1) -> /EN_-3v3
- U7 pad 9: Net-(Cin4-Pad1) -> /EN_-3v3
Routing:
- net /EN_+2v5: track 0.00 -> 7.18 mm
- net /Va: track 0.00 -> 6.94 mm
- net /GND_1v8: track 0.00 -> 4.37 mm
- net /GND_3v3: track 3.85 -> 7.82 mm, vias 0 -> 10
- net /Vafb: track 0.00 -> 3.10 mm
- net /Vreg: track 0.00 -> 1.85 mm
- net /EN_-3v3: track 0.00 -> 1.42 mm
- net /EN_-2v5: track 0.00 -> 1.32 mm
- added copper zone on B.Cu, net (none)
- added copper zone on F.Cu, net /+1v8
- added copper zone on F.Cu, net /+2v5
- added copper zone on F.Cu, net /-1v8
- added copper zone on F.Cu, net /-3v3
- added copper zone on F.Cu, net /EN_+1v8
- added copper zone on F.Cu, net /EN_+2v5
- added copper zone on F.Cu, net /EN_-1v8
- added copper zone on F.Cu, net /EN_-3v3
- added copper zone on B.Cu, net /GND_3v3
- added copper zone on F.Cu, net Net-(J18-Pin_3)
Other:
- board text added: "+"
- board text added: "+Vin"
- board text added: "-"
- board text added: "-Vin"
- board text added: "Bipolar power supply 0x00 Something About Electronics SE/LV 2023"
