File: Hardware/B_PSU_0x00.kicad_sch (KiCad schematic)
At the start: 82 parts, among them J1 Conn_01x03, J10 Conn_01x02, J11 Conn_01x03, J12 Conn_01x03, J13 Conn_01x03, J14 Conn_01x02, J15 Conn_01x02, J16 Conn_01x02, J17 Conn_01x02, J18 Conn_01x03, J19 Conn_01x03, J2 Conn_01x02, J20 Conn_01x03, J21 Conn_01x03, J22 Conn_01x03, J23 Conn_01x02, J24 Conn_01x02, J25 Conn_01x02, J26 Conn_01x02, J27 Conn_01x03, J28 Conn_01x03, J3 Conn_01x03, J4 Conn_01x03, J5 Conn_01x03, J6 Conn_01x03, J7 Conn_01x02, J8 Conn_01x02, J9 Conn_01x02, U1 ADP5070AREZ, U2 ADP7118WAUJZ-5.0, U3 ADP7118AUJZ-3.3-R7, U4 ADP7142AUJZ-1.8, U5 ADP7118AUJZ-2.5-R7, U6 ADP7182ACPZ-5.0-R7, U7 ADP7183ACPZN3.3-R7, U8 ADP7182ACPZN-2.5R7, U9 ADP7182AUJZ-1.8

Commit message: cleaned up layout
Parts:
- U1: footprint Package_SO:ETSSOP-20-1EP_4.4x6.5mm_P0.65mm_EP3x4.2mm -> Package_SO:HSOP-20-1EP_11.0x15.9mm_P1.27mm_SlugDown
Changed lines of the file:
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@@
     (property "Reference" "U1" (id 0) (at 111.76 38.9382 0))
     (property "Value" "ADP5070AREZ" (id 1) (at 111.76 41.2496 0))
-    (property "Footprint" "Package_SO:ETSSOP-20-1EP_4.4x6.5mm_P0.65mm_EP3x4.2mm" (id 2) (at 113.03 91.44 0)
+    (property "Footprint" "Package_SO:HSOP-20-1EP_11.0x15.9mm_P1.27mm_SlugDown" (id 2) (at 113.03 91.44 0)
       (effects (font (size 1.27 1.27)) hide)
     )
@@
     )
     (path "/00000000-0000-0000-0000-000062a12470"
-      (reference "U1") (unit 1) (value "ADP5070AREZ") (footprint "Package_SO:ETSSOP-20-1EP_4.4x6.5mm_P0.65mm_EP3x4.2mm")
+      (reference "U1") (unit 1) (value "ADP5070AREZ") (footprint "Package_SO:HSOP-20-1EP_11.0x15.9mm_P1.27mm_SlugDown")
     )
     (path "/00000000-0000-0000-0000-000062ec2d4d"

Commit message: changed the layout and the size of the PCB
Parts:
- removed J11, J3, J4, J5: Conn_01x03, Connector_PinHeader_2.54mm:PinHeader_1x03_P2.54mm_Vertical, symbol Connector_Generic:Conn_01x03
- U1: footprint Package_SO:HSOP-20-1EP_11.0x15.9mm_P1.27mm_SlugDown -> Package_SO:ETSSOP-20-1EP_4.4x6.5mm_P0.65mm_EP3x4.2mm
- U4: footprint Package_TO_SOT_SMD:TSOT-23-5_HandSoldering -> Package_TO_SOT_SMD:TSOT-23-5
Connections:
- net Vin_+1v8 is gone; now on net EN_+1v8: J16.1 (Pin_1)
- net Vin_+2v5 is gone; now on net EN_+2v5: J17.1 (Pin_1)
- net Vin_+3v3 is gone; now on net EN_+3v3: J9.1 (Pin_1)
- net Vin_+5v is gone; now on net EN_+5v: J7.1 (Pin_1)
- net Vin_-1v8 is gone; now on net EN_-1v8: J8.1 (Pin_1)
- net Vin_-2v5 is gone; now on net EN_-2v5: J15.1 (Pin_1)
- net Vin_-3v3 is gone; now on net EN_-3v3: J10.1 (Pin_1)
- net Vin_-5v is gone; now on net EN_-5v: J2.1 (Pin_1)
- net GND_1v8: now also Cin8.2, Cin9.1, Cout7.2, Cout8.1, J13.2 (Pin_2), J21.2 (Pin_2), J24.2 (Pin_2), U4.2 (GND), U9.1 (GND)
- net GND_2v5: now also Cin5.2, Cin6.2, Cout5.2, Cout6.1, J18.2 (Pin_2), J22.2 (Pin_2), J26.2 (Pin_2), U5.2 (GND), U8.5 (GND)
- net GND_3v3: now also Ca1.2, Cin3.2, Cin4.2, Cout3.2, Cout4.1, Creg1.2, J12.2 (Pin_2), J19.2 (Pin_2), J25.2 (Pin_2), U3.2 (GND), U7.6 (GND)
- net GND_5v: now also Cin2.2, Cin7.1, Cout10.1, Cout9.2, J20.2 (Pin_2), J23.2 (Pin_2), J6.2 (Pin_2), U2.2 (GND), U6.6 (GND)
Other:
- moved on the sheet: Cin8, U4

Commit message: small updates
Other:
- moved on the sheet: J2, J23, J7
Changed lines of the file:
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@@
   (junction (at 375.92 210.82) (diameter 0) (color 0 0 0 0)
   )
-  (junction (at 96.52 259.08) (diameter 0) (color 0 0 0 0)
+  (junction (at 105.41 259.08) (diameter 0) (color 0 0 0 0)
   )
   (junction (at 381 210.82) (diameter 0) (color 0 0 0 0)
@@
   (junction (at 213.36 232.41) (diameter 0) (color 0 0 0 0)
   )
-  (junction (at 130.81 219.71) (diameter 0) (color 0 0 0 0)
+  (junction (at 105.41 219.71) (diameter 0) (color 0 0 0 0)
   )
   (junction (at 285.75 199.39) (diameter 0) (color 0 0 0 0)
@@
   (junction (at 290.83 218.44) (diameter 0) (color 0 0 0 0)
   )
-  (junction (at 128.27 219.71) (diameter 0) (color 0 0 0 0)
+  (junction (at 102.87 219.71) (diameter 0) (color 0 0 0 0)
   )
   (junction (at 370.84 124.46) (diameter 0) (color 0 0 0 0)
@@
   (junction (at 335.28 33.02) (diameter 0) (color 0 0 0 0)
   )
-  (junction (at 83.82 237.49) (diameter 0) (color 0 0 0 0)
+  (junction (at 105.41 245.11) (diameter 0) (color 0 0 0 0)
   )
   (junction (at 372.11 80.01) (diameter 0) (color 0 0 0 0)
@@
   (junction (at 200.66 214.63) (diameter 0) (color 0 0 0 0)
   )
-  (junction (at 81.28 237.49) (diameter 0) (color 0 0 0 0)
+  (junction (at 102.87 245.11) (diameter 0) (color 0 0 0 0)
   )
   (junction (at 132.08 245.11) (diameter 0) (color 0 0 0 0)
@@
   (junction (at 391.16 137.16) (diameter 0) (color 0 0 0 0)
   )
-  (junction (at 93.98 259.08) (diameter 0) (color 0 0 0 0)
+  (junction (at 102.87 259.08) (diameter 0) (color 0 0 0 0)
   )
   (junction (at 156.21 260.35) (diameter 0) (color 0 0 0 0)
@@
     (stroke (width 0) (type default) (color 0 0 0 0))
   )
-  (wire (pts (xy 128.27 219.71) (xy 115.57 219.71))
+  (wire (pts (xy 102.87 219.71) (xy 90.17 219.71))
     (stroke (width 0) (type default) (color 0 0 0 0))
   )
@@
     (stroke (width 0) (type default) (color 0 0 0 0))
   )
-  (wire (pts (xy 81.28 259.08) (xy 78.74 256.54))
+  (wire (pts (xy 90.17 259.08) (xy 87.63 256.54))
     (stroke (width 0) (type default) (color 0 0 0 0))
   )
@@
     (stroke (width 0) (type default) (color 0 0 0 0))
   )
-  (wire (pts (xy 83.82 237.49) (xy 81.28 237.49))
+  (wire (pts (xy 105.41 245.11) (xy 102.87 245.11))
     (stroke (width 0) (type default) (color 0 0 0 0))
   )
@@
     (stroke (width 0) (type default) (color 0 0 0 0))
   )
-  (wire (pts (xy 130.81 219.71) (xy 128.27 219.71))
+  (wire (pts (xy 105.41 219.71) (xy 102.87 219.71))
     (stroke (width 0) (type default) (color 0 0 0 0))
   )
@@
     (stroke (width 0) (type default) (color 0 0 0 0))
   )
-  (wire (pts (xy 81.28 237.49) (xy 72.39 237.49))
+  (wire (pts (xy 102.87 245.11) (xy 93.98 245.11))
     (stroke (width 0) (type default) (color 0 0 0 0))
   )
@@
     (stroke (width 0) (type default) (color 0 0 0 0))
   )
-  (wire (pts (xy 115.57 219.71) (xy 113.03 217.17))
+  (wire (pts (xy 90.17 219.71) (xy 87.63 217.17))
     (stroke (width 0) (type default) (color 0 0 0 0))
   )
@@
     (stroke (width 0) (type default) (color 0 0 0 0))
   )
-  (wire (pts (xy 130.81 219.71) (xy 138.43 219.71))
+  (wire (pts (xy 105.41 219.71) (xy 138.43 219.71))
     (stroke (width 0) (type default) (color 0 0 0 0))
   )
@@
     (stroke (width 0) (type default) (color 0 0 0 0))
   )
-  (wire (pts (xy 72.39 237.49) (xy 69.85 236.22))
+  (wire (pts (xy 93.98 245.11) (xy 91.44 243.84))
     (stroke (width 0) (type default) (color 0 0 0 0))
   )
@@
     (stroke (width 0) (type default) (color 0 0 0 0))
   )
-  (wire (pts (xy 96.52 259.08) (xy 93.98 259.08))
+  (wire (pts (xy 105.41 259.08) (xy 102.87 259.08))
     (stroke (width 0) (type default) (color 0 0 0 0))
   )
@@
     (stroke (width 0) (type default) (color 0 0 0 0))
   )
-  (wire (pts (xy 83.82 245.11) (xy 83.82 237.49))
-    (stroke (width 0) (type default) (color 0 0 0 0))
-  )
   (wire (pts (xy 381 222.25) (xy 384.81 222.25))
     (stroke (width 0) (type default) (color 0 0 0 0))
@@
     (stroke (width 0) (type default) (color 0 0 0 0))
   )
-  (wire (pts (xy 83.82 245.11) (xy 132.08 245.11))
+  (wire (pts (xy 105.41 245.11) (xy 132.08 245.11))
     (stroke (width 0) (type default) (color 0 0 0 0))
   )
@@
     (stroke (width 0) (type default) (color 0 0 0 0))
   )
-  (wire (pts (xy 93.98 259.08) (xy 81.28 259.08))
+  (wire (pts (xy 102.87 259.08) (xy 90.17 259.08))
     (stroke (width 0) (type default) (color 0 0 0 0))
   )
@@
     (stroke (width 0) (type default) (color 0 0 0 0))
   )
-  (wire (pts (xy 96.52 259.08) (xy 132.08 259.08))
+  (wire (pts (xy 105.41 259.08) (xy 132.08 259.08))
     (stroke (width 0) (type default) (color 0 0 0 0))
   )
@@
     (effects (font (size 1.27 1.27)) (justify left bottom))
   )
-  (label "GND_5v" (at 69.85 236.22 0)
+  (label "GND_5v" (at 91.44 243.84 0)
     (effects (font (size 1.27 1.27)) (justify left bottom))
   )
@@
     (effects (font (size 1.27 1.27)) (justify left bottom))
   )
-  (label "Vin_-5v" (at 78.74 256.54 0)
+  (label "Vin_-5v" (at 87.63 256.54 0)
     (effects (font (size 1.27 1.27)) (justify left bottom))
   )
@@
     (effects (font (size 1.27 1.27)) (justify left bottom))
   )
-  (label "Vin_+5v" (at 113.03 217.17 0)
+  (label "Vin_+5v" (at 87.63 217.17 0)
     (effects (font (size 1.27 1.27)) (justify left bottom))
   )
@@
     (pin "2")
   )
-  (symbol (lib_id "power:GNDA") (at 154.94 107.95 0) (unit 1)
-    (in_bom yes) (on_board yes)
-    (property "Reference" "#PWR0115" (id 0) (at 154.94 114.3 0)
-      (effects (font (size 1.27 1.27)) hide)
-    )
-    (property "Value" "GNDA" (id 1) (at 155.067 112.3442 0))
-    (property "Footprint" "" (id 2) (at 154.94 107.95 0)
-      (effects (font (size 1.27 1.27)) hide)
-    )
-    (property "Datasheet" "" (id 3) (at 154.94 107.95 0)
-      (effects (font (size 1.27 1.27)) hide)
-    )
-    (pin "1")
-  )
   (symbol (lib_id "power:GNDREF") (at 128.27 93.98 0) (unit 1)
     (in_bom yes) (on_board yes)
@@
     (pin "2")
   )
-  (symbol (lib_id "Connector_Generic:Conn_01x02") (at 128.27 214.63 90) (unit 1)
+  (symbol (lib_id "Connector_Generic:Conn_01x02") (at 102.87 214.63 90) (unit 1)
     (in_bom yes) (on_board yes)
-    (property "Reference" "J7" (id 0) (at 133.0452 215.5444 90)
+    (property "Reference" "J7" (id 0) (at 107.6452 215.5444 90)
       (effects (font (size 1.27 1.27)) (justify right))
     )
-    (property "Value" "Conn_01x02" (id 1) (at 133.0452 217.8558 90)
+    (property "Value" "Conn_01x02" (id 1) (at 107.6452 217.8558 90)
       (effects (font (size 1.27 1.27)) (justify right))
     )
-    (property "Footprint" "Connector_PinHeader_2.54mm:PinHeader_1x02_P2.54mm_Vertical" (id 2) (at 128.27 214.63 0)
+    (property "Footprint" "Connector_PinHeader_2.54mm:PinHeader_1x02_P2.54mm_Vertical" (id 2) (at 102.87 214.63 0)
       (effects (font (size 1.27 1.27)) hide)
     )
-    (property "Datasheet" "~" (id 3) (at 128.27 214.63 0)
+    (property "Datasheet" "~" (id 3) (at 102.87 214.63 0)
       (effects (font (size 1.27 1.27)) hide)
     )
@@
     (pin "2")
   )
-  (symbol (lib_id "Connector_Generic:Conn_01x02") (at 93.98 254 90) (unit 1)
+  (symbol (lib_id "Connector_Generic:Conn_01x02") (at 102.87 254 90) (unit 1)
     (in_bom yes) (on_board yes)
-    (property "Reference" "J2" (id 0) (at 98.7552 254.9144 90)
+    (property "Reference" "J2" (id 0) (at 107.6452 254.9144 90)
       (effects (font (size 1.27 1.27)) (justify right))
     )
-    (property "Value" "Conn_01x02" (id 1) (at 98.7552 257.2258 90)
+    (property "Value" "Conn_01x02" (id 1) (at 107.6452 257.2258 90)
       (effects (font (size 1.27 1.27)) (justify right))
     )
-    (property "Footprint" "Connector_PinHeader_2.54mm:PinHeader_1x02_P2.54mm_Vertical" (id 2) (at 93.98 254 0)
+    (property "Footprint" "Connector_PinHeader_2.54mm:PinHeader_1x02_P2.54mm_Vertical" (id 2) (at 102.87 254 0)
       (effects (font (size 1.27 1.27)) hide)
     )
-    (property "Datasheet" "~" (id 3) (at 93.98 254 0)
+    (property "Datasheet" "~" (id 3) (at 102.87 254 0)
       (effects (font (size 1.27 1.27)) hide)
     )
@@
     (pin "2")
   )
-  (symbol (lib_id "Connector_Generic:Conn_01x02") (at 81.28 232.41 90) (unit 1)
+  (symbol (lib_id "Connector_Generic:Conn_01x02") (at 102.87 240.03 90) (unit 1)
     (in_bom yes) (on_board yes)
-    (property "Reference" "J23" (id 0) (at 86.0552 233.3244 90)
+    (property "Reference" "J23" (id 0) (at 107.6452 240.9444 90)
       (effects (font (size 1.27 1.27)) (justify right))
     )
-    (property "Value" "Conn_01x02" (id 1) (at 86.0552 235.6358 90)
+    (property "Value" "Conn_01x02" (id 1) (at 107.6452 243.2558 90)
       (effects (font (size 1.27 1.27)) (justify right))
     )
-    (property "Footprint" "Connector_PinHeader_2.54mm:PinHeader_1x02_P2.54mm_Vertical" (id 2) (at 81.28 232.41 0)
+    (property "Footprint" "Connector_PinHeader_2.54mm:PinHeader_1x02_P2.54mm_Vertical" (id 2) (at 102.87 240.03 0)
       (effects (font (size 1.27 1.27)) hide)
     )
-    (property "Datasheet" "~" (id 3) (at 81.28 232.41 0)
+    (property "Datasheet" "~" (id 3) (at 102.87 240.03 0)
       (effects (font (size 1.27 1.27)) hide)
     )
@@
       (reference "#PWR0114") (unit 1) (value "GNDA") (footprint "")
     )
-    (path "/00000000-0000-0000-0000-0000633fa006"
-      (reference "#PWR0115") (unit 1) (value "GNDA") (footprint "")
-    )
     (path "/00000000-0000-0000-0000-0000634312c2"

Commit message: small updates
Connections:
- net -2v5: no longer Cout6.2, J18.3 (Pin_3), J22.3 (Pin_3), U8.1 (Vout)
- net -3v3: no longer Cout4.2, J12.3 (Pin_3), J19.3 (Pin_3), U7.1 (VOUT), U7.2 (SENSE)
- new net: Cout4.2, J12.3 (Pin_3), J19.3 (Pin_3), U7.1 (VOUT), U7.2 (SENSE)
- new net: Cout6.2, J18.3 (Pin_3), J22.3 (Pin_3), U8.1 (Vout)

Commit message: 0x00 version and revision files for manufacturing
Connections:
- net -3v3: now also Cout4.2, J12.3 (Pin_3), J19.3 (Pin_3), U7.1 (VOUT), U7.2 (SENSE)
- net Va: now reaches Ca1.1, Cafb1.1, U7.3 (VA)
- net Vafb: now reaches Cafb1.2, U7.4 (VAFB)
- net Vreg: now reaches Creg1.1, U7.7 (VREG)
Other:
- company: (none) -> Something About Electronics
- title: (none) -> Multi rail Bipolar low noise power supply
- moved on the sheet: Ca1
